Commit message: Add inertia and contact tags on some urdf in multicontact subfolder (required by pybullet)

File: urdf/multicontact/ground.urdf (robot description, URDF)
Before this commit: robot chair, 1 links, 0 joints
Links:
- removed link base_link
- added link ground_link, mass .0; collision mesh filename=package://hpp_environments/meshes/multicontact/ground.stl; visual mesh filename=package://hpp_environments/meshes/multicontact/ground.stl

File: urdf/multicontact/ori_plinth.urdf (robot description, URDF)
Before this commit: robot ori_plinth, 1 links, 0 joints
Links:
- link base_link: mass None -> .0

File: urdf/multicontact/plateforme_surfaces.urdf (robot description, URDF)
Before this commit: robot stair_bauzil, 1 links, 0 joints
Links:
- removed link base_link
- added link plateforme_link, mass .0; collision mesh filename=package://hpp_environments/meshes/multicontact/plateforme_s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; visual mesh filename=package://hpp_environments/meshes/multicontact/plateforme_s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

File: urdf/multicontact/slalom_debris.urdf (robot description, URDF)
Before this commit: robot chair, 1 links, 0 joints
Links:
- removed link base_link
- added link slalom_link, mass .0; collision mesh filename=package://hpp_environments/meshes/multicontact/slalom_debri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; visual mesh filename=package://hpp_environments/meshes/multicontact/slalom_debri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
